File: Arduino Mega V1/ic_mega(v1).brd (EAGLE design)
At the start: 99.1 x 52.8 mm, 45 parts, among them IC1 TL071P, IC2 LM7805, J1 F-2X07-79107_M, J5 F-1X02-SIP-100-32, J6 DAC, U2 INA333AIDRGT, U3 INA333AIDRGT, U4 INA333AIDRGT, U5 INA333AIDRGT

Commit message: versao final 1
Connections:
- net GNDA: now also C2.2, U3.4
- net VSS: no longer C2.2, U3.4
Routing:
- net GNDA: track 21.5 -> 36.1 mm, vias 0 -> 1
- net VSS: track 79.8 -> 75.8 mm, vias 1 -> 0
Changed lines of the file:
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@@
 <wire x1="71.374" y1="30.988" x2="69.85" y2="29.464" width="0.254" layer="16"/>
 <wire x1="69.85" y1="29.464" x2="65.532" y2="29.464" width="0.254" layer="16"/>
+<contactref element="C2" pad="2"/>
+<contactref element="U3" pad="4"/>
+<wire x1="35.941" y1="27.94" x2="35.306" y2="27.94" width="0.254" layer="1"/>
+<wire x1="35.306" y1="27.94" x2="34.798" y2="27.432" width="0.254" layer="1"/>
+<via x="34.798" y="27.432" extent="1-16" drill="0.35"/>
+<wire x1="34.798" y1="27.432" x2="35.052" y2="27.178" width="0.254" layer="16"/>
+<wire x1="35.052" y1="27.178" x2="35.052" y2="24.892" width="0.254" layer="16"/>
+<wire x1="35.052" y1="24.892" x2="34.036" y2="23.876" width="0.254" layer="1"/>
+<wire x1="34.036" y1="23.876" x2="24.892" y2="23.876" width="0.254" layer="1"/>
 <wire x1="87.772" y1="8.652" x2="94.996" y2="7.874" width="0" layer="19" extent="1-1"/>
 <wire x1="52.705" y1="18.542" x2="63.754" y2="17.272" width="0" layer="19" extent="1-1"/>
@@
 <contactref element="R5" pad="1"/>
 <contactref element="B1" pad="3.3V"/>
-<contactref element="C2" pad="2"/>
-<contactref element="U3" pad="4"/>
 <wire x1="28.829" y1="5.969" x2="33.401" y2="5.969" width="0.254" layer="16"/>
 <wire x1="33.401" y1="5.969" x2="36.576" y2="2.794" width="0.254" layer="16"/>
-<wire x1="35.941" y1="27.94" x2="35.306" y2="27.94" width="0.254" layer="1"/>
-<wire x1="35.306" y1="27.94" x2="34.798" y2="27.432" width="0.254" layer="1"/>
-<via x="34.798" y="27.432" extent="1-16" drill="0.35"/>
-<wire x1="34.798" y1="27.432" x2="35.052" y2="27.178" width="0.254" layer="16"/>
-<wire x1="35.052" y1="27.178" x2="35.052" y2="24.892" width="0.254" layer="16"/>
 <wire x1="45.958" y1="22.638" x2="44.958" y2="23.638" width="0.254" layer="16"/>
 <wire x1="44.958" y1="29.638" x2="43.958" y2="30.638" width="0.254" layer="16"/>
@@
 <wire x1="61.468" y1="15.748" x2="61.468" y2="40.005" width="0.254" layer="1"/>
 <wire x1="61.468" y1="40.005" x2="59.69" y2="41.783" width="0.254" layer="1"/>
-<wire x1="35.052" y1="24.892" x2="43.958" y2="30.638" width="0" layer="19" extent="1-1"/>
-<wire x1="43.958" y1="30.638" x2="59.69" y2="41.783" width="0" layer="19" extent="1-1"/>
+<wire x1="59.69" y1="41.783" x2="43.958" y2="30.638" width="0" layer="19" extent="1-1"/>
 </signal>
 <signal name="N$15">
